File: TouchscreenAdapter/TouchscreenAdapter.sch (KiCad schematic (older format))
At the start: 61 parts, among them J1 Conn_01x40_Male, J2 Conn_01x04, J3 Barrel_Jack, J4 Conn_01x04, J5 Conn_01x02_Male, J6 Conn_01x02_Male, J7 Conn_02x10_Odd_Even, J8 Conn_01x02_Male, Q1 Q_PMOS_DGS, U1 LT1945EMS-PBF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

Commit message: Updated Resistor Values
Parts:
- R14: value R -> 680k
- R15, R16: value R -> 100k
- R17: value R -> 330k
- R18: value R -> 270k
- R19: value R -> 20k
- U1: symbol LT1945EMS-PBF:LT1945EMS-PBF -> TouchscreenAdapter-rescue:LT1945EMS-PBF-LT1945EMS-PBF
Changed lines of the file:
@@
 EESchema Schematic File Version 4
 LIBS:TouchscreenAdapter-cache
-EELAYER 26 0
+EELAYER 29 0
 EELAYER END
 $Descr A3 16535 11693
@@
 $EndBitmap
 $Comp
-L LT1945EMS-PBF:LT1945EMS-PBF U1
+L TouchscreenAdapter-rescue:LT1945EMS-PBF-LT1945EMS-PBF U1
 U 1 1 5CA2B903
 P 8000 6100
@@
 P 8700 4750
 F 0 "R14" H 8770 4796 50  0000 L CNN
-F 1 "R" H 8770 4705 50  0000 L CNN
+F 1 "680k" H 8770 4705 50  0000 L CNN
 F 2 "Resistor_SMD:R_0805_2012Metric_Pad1.15x1.40mm_HandSolder" V 8630 4750 50  0001 C CNN
 F 3 "~" H 8700 4750 50  0001 C CNN
@@
 P 9150 5050
 F 0 "R15" V 8943 5050 50  0000 C CNN
-F 1 "R" V 9034 5050 50  0000 C CNN
+F 1 "100k" V 9034 5050 50  0000 C CNN
 F 2 "Resistor_SMD:R_0805_2012Metric_Pad1.15x1.40mm_HandSolder" V 9080 5050 50  0001 C CNN
 F 3 "~" H 9150 5050 50  0001 C CNN
@@
 P 10400 4700
 F 0 "R17" H 10470 4746 50  0000 L CNN
-F 1 "R" H 10470 4655 50  0000 L CNN
+F 1 "330k" H 10470 4655 50  0000 L CNN
 F 2 "Resistor_SMD:R_0805_2012Metric_Pad1.15x1.40mm_HandSolder" V 10330 4700 50  0001 C CNN
 F 3 "~" H 10400 4700 50  0001 C CNN
@@
 P 9950 5000
 F 0 "R16" V 9743 5000 50  0000 C CNN
-F 1 "R" V 9834 5000 50  0000 C CNN
+F 1 "100k" V 9834 5000 50  0000 C CNN
 F 2 "Resistor_SMD:R_0805_2012Metric_Pad1.15x1.40mm_HandSolder" V 9880 5000 50  0001 C CNN
 F 3 "~" H 9950 5000 50  0001 C CNN
@@
 P 12250 4600
 F 0 "R18" H 12320 4646 50  0000 L CNN
-F 1 "R" H 12320 4555 50  0000 L CNN
+F 1 "270k" H 12320 4555 50  0000 L CNN
 F 2 "Resistor_SMD:R_0805_2012Metric_Pad1.15x1.40mm_HandSolder" V 12180 4600 50  0001 C CNN
 F 3 "~" H 12250 4600 50  0001 C CNN
@@
 P 12250 5650
 F 0 "R19" H 12320 5696 50  0000 L CNN
-F 1 "R" H 12320 5605 50  0000 L CNN
+F 1 "20k" H 12320 5605 50  0000 L CNN
 F 2 "Resistor_SMD:R_0805_2012Metric_Pad1.15x1.40mm_HandSolder" V 12180 5650 50  0001 C CNN
 F 3 "~" H 12250 5650 50  0001 C CNN
